File: KiCAD/forthEx.sch (KiCad schematic (older format))
At the start: 52 parts, among them CON1 SD_Card, CON2 BARREL_JACK 2,1mm, J1 RCA_JACK, J2 RCA_JACK, J3 USB-A_F, J4 miniDIN-6, P1 ICSP, Q1 2N3906, Q2 2N3904, SW1 Power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

Commit message: modification circuit
l'interface avec le clavier est maintenant assuré par un second MCU PIC12F1572. Logiciel modifié en conséquence. le code pour l'interface clavier est dans un projet séparé sur https://github.com/picatout/ps2_rs232
Parts:
- removed J3: USB-A_F, symbol USB-A_F
- removed J4: miniDIN-6, ~, symbol PS/2
- removed R14: 10K, ~, symbol R-RESCUE-forthEx
- added D4, D6: 1N4148, symbol D
- added J3: RJ12, symbol RJ12
- added R14: 10K, symbol R
- added R18, R23: 10K, ~, symbol R-RESCUE-forthEx
Connections:
- net labels removed: KBCLK, KBDAT
- wire segments 147 -> 156
- no-connect marks 1 -> 6
Other:
- note added: "ForthEx\nForth explorer computer\nCopyright, Jacques Deschenes, 2016,2017\nlicence: CC-BY_SA-V3.0"
- note added: "forthex"
- note removed: "connecteur clavier\n"
- note removed: "option 1"
- note removed: "option 2"
- moved on the sheet: C2, D1, D3, J1, Q1, Q2, R1, R10, R2, R3, R4, R8

Commit message: ajout code SDCard
Parts:
- added D7: 1N4148, symbol D
- added R24, R25: 10K, ~, symbol R-RESCUE-forthEx
Connections:
- net +3,3V: now also C11.1, P1.2, R13.2, R18.2, R23.2, U3.28 (Vdd), D7.1 (K), R24.2, R25.2
- net CD: now also R24.1
- net ~SS3: now also R25.1
- net at C7.1, R6.1, R7.1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: now also D7.2 (A)
Changed lines of the file:
@@
 	-1   0    0    1
 $EndComp
-Text GLabel 6850 3450 2    39   Input ~ 0
+Text GLabel 7700 3450 2    39   Input ~ 0
 CD
 Text GLabel 750  4200 0    39   Input ~ 0
@@
 Text GLabel 2550 4000 2    39   Input ~ 0
 +3,3V
-Text GLabel 5200 3550 0    39   Input ~ 0
+Text GLabel 4850 3550 0    39   Input ~ 0
 ~SS3
 Text GLabel 2550 3900 2    39   Input ~ 0
@@
 Connection ~ 2400 850
 Wire Wire Line
-	6850 3450 6700 3450
+	6700 3450 7700 3450
 Wire Wire Line
 	2750 3800 2750 4650
@@
 	8350 1700 8550 1700
 Wire Wire Line
-	3050 2400 3900 2400
-Wire Wire Line
-	3950 2400 7550 2400
+	3050 2400 7700 2400
 Wire Wire Line
 	7900 3250 7900 3200
@@
 	5350 1400 8550 1400
 Connection ~ 5200 2950
+$Comp
+L R-RESCUE-forthEx R24
+U 1 1 587A4268
+P 7700 2850
+F 0 "R24" V 7780 2850 40  0000 C CNN
+F 1 "10K" V 7707 2851 40  0000 C CNN
+F 2 "~" V 7630 2850 30  0000 C CNN
+F 3 "~" H 7700 2850 30  0000 C CNN
+	1    7700 2850
+	-1   0    0    1
+$EndComp
+Wire Wire Line
+	7700 2400 7700 2600
+Wire Wire Line
+	7700 3450 7700 3100
+$Comp
+L R-RESCUE-forthEx R25
+U 1 1 587AB52E
+P 4400 2650
+F 0 "R25" V 4480 2650 40  0000 C CNN
+F 1 "10K" V 4407 2651 40  0000 C CNN
+F 2 "~" V 4330 2650 30  0000 C CNN
+F 3 "~" H 4400 2650 30  0000 C CNN
+	1    4400 2650
+	-1   0    0    1
+$EndComp
+Connection ~ 4400 2400
+Wire Wire Line
+	4400 2900 4850 2900
+Wire Wire Line
+	4850 2900 4850 3550
+Wire Wire Line
+	4850 3550 5200 3550
+$Comp
+L D D7
+U 1 1 587CE66F
+P 3650 2800
+F 0 "D7" H 3650 2900 50  0000 C CNN
+F 1 "1N4148" H 3650 2700 50  0000 C CNN
+F 2 "" H 3650 2800 50  0000 C CNN
+F 3 "" H 3650 2800 50  0000 C CNN
+	1    3650 2800
+	0    1    1    0
+$EndComp
+Wire Wire Line
+	3650 2650 3650 2400
+Connection ~ 3650 2400
+Wire Wire Line
+	3650 2950 3650 3100
+Connection ~ 3650 3100
 $EndSCHEMATC

Commit message: réorganisation projet
Changed lines of the file:
@@
 NoConn ~ 750  5850
-$Comp
-L R-RESCUE-forthEx R18
-U 1 1 5873EBF4
-P 7000 2950
-F 0 "R18" V 7080 2950 40  0000 C CNN
-F 1 "10K" V 7007 2951 40  0000 C CNN
-F 2 "~" V 6930 2950 30  0000 C CNN
-F 3 "~" H 7000 2950 30  0000 C CNN
-	1    7000 2950
-	-1   0    0    1
-$EndComp
 $Comp
 L R R14
@@
 	8350 1700 8550 1700
 Wire Wire Line
-	3050 2400 7700 2400
+	3050 2400 8450 2400
 Wire Wire Line
 	7900 3250 7900 3200
@@
 	5200 6850 5600 6850
 Wire Wire Line
-	6700 3350 8250 3350
-Wire Wire Line
 	4850 4150 4850 4250
 Connection ~ 4850 4250
 Wire Wire Line
 	5150 4150 5200 4150
-Wire Wire Line
-	7000 3350 7000 3200
 $Comp
 L GND #PWR17
@@
 	1    0    0    -1
 $EndComp
-$Comp
-L D D6
-U 1 1 58740C49
-P 8250 3050
-F 0 "D6" H 8250 3150 50  0000 C CNN
-F 1 "1N4148" H 8250 2950 50  0000 C CNN
-F 2 "" H 8250 3050 50  0000 C CNN
-F 3 "" H 8250 3050 50  0000 C CNN
-	1    8250 3050
-	0    1    1    0
-$EndComp
-Wire Wire Line
-	8250 3350 8250 3200
-Connection ~ 7000 3350
-Wire Wire Line
-	8250 2900 8250 2100
 Wire Wire Line
 	8250 2100 8550 2100
@@
 	3650 2950 3650 3100
 Connection ~ 3650 3100
+$Comp
+L D D6
+U 1 1 58897471
+P 8250 3050
+F 0 "D6" H 8250 3150 50  0000 C CNN
+F 1 "1N4148" H 8250 2950 50  0000 C CNN
+F 2 "" H 8250 3050 50  0000 C CNN
+F 3 "" H 8250 3050 50  0000 C CNN
+	1    8250 3050
+	0    1    1    0
+$EndComp
+Wire Wire Line
+	8250 2100 8250 2900
+Wire Wire Line
+	8250 3200 8250 3350
+Wire Wire Line
+	6700 3350 8450 3350
+$Comp
+L R-RESCUE-forthEx R18
+U 1 1 588977AF
+P 8450 2850
+F 0 "R18" V 8530 2850 40  0000 C CNN
+F 1 "10K" V 8457 2851 40  0000 C CNN
+F 2 "~" V 8380 2850 30  0000 C CNN
+F 3 "~" H 8450 2850 30  0000 C CNN
+	1    8450 2850
+	-1   0    0    1
+$EndComp
+Wire Wire Line
+	8450 2400 8450 2600
+Connection ~ 7700 2400
+Wire Wire Line
+	8450 3350 8450 3100
+Connection ~ 8250 3350
 $EndSCHEMATC
