File: KiCAD/ForthEx_s/alim_5neg.sch (KiCad schematic (older format))
At the start: 11 parts, among them U7 TLC555

Commit message: travail sur documentation
Parts:
- gave numbers to parts that had none: 1
Changed lines of the file:
@@
 $Descr A4 11693 8268
 encoding utf-8
-Sheet 3 3
+Sheet 3 4
 Title ""
 Date ""
@@
 $EndComp
 $Comp
-L GND #PWR39
+L GND #PWR35
 U 1 1 593B2BFD
 P 4550 2850
-F 0 "#PWR39" H 4550 2600 50  0001 C CNN
+F 0 "#PWR35" H 4550 2600 50  0001 C CNN
 F 1 "GND" H 4550 2700 50  0000 C CNN
 F 2 "" H 4550 2850 50  0001 C CNN
@@
 	4550 2800 4550 2850
 $Comp
-L GND #PWR40
+L GND #PWR36
 U 1 1 593B2CAB
 P 4650 3500
-F 0 "#PWR40" H 4650 3250 50  0001 C CNN
+F 0 "#PWR36" H 4650 3250 50  0001 C CNN
 F 1 "GND" H 4650 3350 50  0000 C CNN
 F 2 "" H 4650 3500 50  0001 C CNN
@@
 $EndComp
 $Comp
-L GND #PWR42
+L GND #PWR38
 U 1 1 593B2CD7
 P 6550 4250
-F 0 "#PWR42" H 6550 4000 50  0001 C CNN
+F 0 "#PWR38" H 6550 4000 50  0001 C CNN
 F 1 "GND" H 6550 4100 50  0000 C CNN
 F 2 "" H 6550 4250 50  0001 C CNN
@@
 $EndComp
 $Comp
-L GND #PWR41
+L GND #PWR37
 U 1 1 593B2D03
 P 5750 3600
-F 0 "#PWR41" H 5750 3350 50  0001 C CNN
+F 0 "#PWR37" H 5750 3350 50  0001 C CNN
 F 1 "GND" H 5750 3450 50  0000 C CNN
 F 2 "" H 5750 3600 50  0001 C CNN
@@
 $EndComp
 $Comp
-L GND #PWR43
+L GND #PWR39
 U 1 1 593B2D2F
 P 6950 3400
-F 0 "#PWR43" H 6950 3150 50  0001 C CNN
+F 0 "#PWR39" H 6950 3150 50  0001 C CNN
 F 1 "GND" H 6950 3250 50  0000 C CNN
 F 2 "" H 6950 3400 50  0001 C CNN
@@
 $EndComp
 $Comp
-L GND #PWR44
+L GND #PWR40
 U 1 1 593B2D5B
 P 7650 3400
-F 0 "#PWR44" H 7650 3150 50  0001 C CNN
+F 0 "#PWR40" H 7650 3150 50  0001 C CNN
 F 1 "GND" H 7650 3250 50  0000 C CNN
 F 2 "" H 7650 3400 50  0001 C CNN
@@
 $EndComp
 $Comp
-L C C?
+L C C18
 U 1 1 593B2E41
 P 4700 2650
-F 0 "C?" H 4725 2750 50  0000 L CNN
+F 0 "C18" H 4725 2750 50  0000 L CNN
 F 1 "100nF" H 4725 2550 50  0000 L CNN
 F 2 "" H 4738 2500 50  0001 C CNN
