File: KiCAD/ForthEx_s/forthEx.sch (KiCad schematic (older format))
At the start: 59 parts, among them CON1 SD_Card, CON2 BARREL_JACK 2,1mm, J1 RCA_JACK, J2 RCA_JACK, J3 RJ12, P1 ICSP, Q1 2N3906, Q2 2N3904, SW1 Power, SW2 reset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

Commit message: travail sur documentation
Parts:
- removed C18: 4,7µF, ~, symbol CAPAPOL
- removed C19: 220µF, ~, symbol CAPAPOL
- removed CON1: SD_Card, 10067847-001, symbol SD_Card
- removed L1: 15µH, symbol L
- removed R25: 10K, ~, symbol R-RESCUE-forthEx
- removed U4: 25LC1024, symbol 23LC512
- added S1: eeprom, symbol conn_f_01x06
Connections:
- net labels added: gnd, miso, mosi, sclk, ~ss1, ~ss2
- net labels removed: +Vsdc, MISO, MOSI, SCLK, ~SS1, ~SS2, ~SS3
- wire segments 168 -> 141
Other:
- note added: "COM"
- note added: "RAM"
